File: test.sch (KiCad schematic (older format))
At the start: 24 parts, among them J1 Conn_01x06_Female, J2 Conn_02x02_Top_Bottom, J3 Conn_02x03_Odd_Even, J4 Conn_01x02, J5 Conn_01x02, J6 Conn_02x02_Top_Bottom, J7 Conn_02x10_Counter_Clockwise, SW1 PTS647SK38SMTR2LFS, U1 PIC32MX340F512H-80I_MR

Commit message: - Reworked schematic with more recognizable symbols, more information, more adherent to FAQ, etc. - Shifted from 4 layer to 2 layer - Removed all micro/hidden vias - Standardized footprints for all resistors and capacitors - Shifted all headers from SMD to througholes - Added more information to silkscreen
Parts:
- removed C1, C3, C6: CL05A104KA5NNNC, mod:CL05A104KA5NNNC, symbol ul_CL05A104KA5NNNC:CL05A104KA5NNNC
- removed C5: CL10A106MQ8NNNC, mod:CL10A106MQ8NNNC, symbol ul_CL10A106MQ8NNNC:CL10A106MQ8NNNC
- added C1, C3, C5: 0.1uF, mod:CL10A106MQ8NNNC, symbol pspice:C
- added C6: 10uF, mod:CL10A106MQ8NNNC, symbol pspice:C
- added R5, R6: 4.7kΩ, mod:ERJ-3EKF10R0V, symbol Device:R_Small_US
- C2, C4: value CL05A104KA5NNNC -> 0.1uF; footprint mod:CL05A104KA5NNNC -> mod:CL10A106MQ8NNNC; symbol ul_CL05A104KA5NNNC:CL05A104KA5NNNC -> pspice:C
- J1: value Conn_01x06_Female -> ICSP; footprint mod:SULLINS_NPPN061BFLD-RC -> mod:01x06
- J2: value Conn_02x02_Top_Bottom -> SPI; footprint mod:969973-2 -> mod:02x02
- J3: value Conn_02x03_Odd_Even -> UART; footprint mod:M20-7870346 -> mod:02x03
- J4: value Conn_01x02 -> 3.3v VDD
- J5: value Conn_01x02 -> VSS
- J6: renamed from J7; value Conn_02x10_Counter_Clockwise -> GPIO Header; footprint mod:NPPC102KFMS-RC -> mod:02x20
- J7: renamed from J6; value Conn_02x02_Top_Bottom -> I2C; footprint mod:969973-2 -> mod:02x02
- R1, R2: footprint mod:RMCF2512JT470R -> mod:ERJ-3EKF10R0V; symbol Device:R -> Device:R_Small_US
- R3: footprint mod:RMCF2512FT10K0 -> mod:ERJ-3EKF10R0V; symbol Device:R -> Device:R_Small_US
- R4: footprint mod:RMCF2512JT10R0 -> mod:ERJ-3EKF10R0V; symbol Device:R -> Device:R_Small_US
- SW1: value PTS647SK38SMTR2LFS -> Reset Button
- TP1: footprint TestPoint:TestPoint_Pad_D1.5mm -> TestPoint:TestPoint_Pad_D1.0mm
- renumbered MK4 to MK3, MK3 to MK4
Connections:
- net labels added: GNDREF
- net labels removed: GND
- wire segments 162 -> 179
- no-connect marks 28 -> 27
Other:
- moved on the sheet: MK2, MK3

Commit message: - Changed board size to 1" by 2" - added 40mil exclusion zone from board edges - changed default trace to 8 mil - changed exclusion to 8 mil - changed power traces to 12 mil - added more descriptive silkscreen
Parts:
- removed MK1, MK2, MK3, MK4: Mounting_Hole_PAD, MountingHole:MountingHole_2.7mm, symbol test-rescue:Mounting_Hole_PAD-Mechanical-test-rescue
- J2, J7: symbol Connector_Generic:Conn_02x02_Top_Bottom -> Connector_Generic:Conn_02x02_Odd_Even; Mfr (none) -> Samtec Inc.; Mfr # (none) -> SSW-102-01-T-D
- J3: Mfr (none) -> Samtec Inc.; Mfr # (none) -> SSW-103-01-T-D
- J4, J5: Mfr (none) -> TE Connectivity AMP Connectors; Mfr # (none) -> RCS-0C
- J6: symbol Connector_Generic:Conn_02x10_Counter_Clockwise -> Connector_Generic:Conn_02x10_Odd_Even; Mfr (none) -> Samtec Inc.; Mfr # (none) -> SSW-110-01-T-D
- SW1: Mfr (none) -> C&K; Mfr # (none) -> PTS647SK38SMTR2LFS
- U1: Mfr (none) -> Microchip Technology; Mfr # (none) -> PIC32MX340F512H-80I/MR
Connections:
- wire segments 179 -> 199
- no-connect marks 27 -> 29

Commit message: - Added 4 User LEDs - Added 1 Power LED - Added 5 68ohm resistors to complement above LEDs - Reshaped board to 1.8"-1.1" - Added pin 52 to / Removed pin 42 from GPIO header (traded an INT for an extra OC/CN) - Reverted changed to corner pads for PIC back to original Microchip pad, just changed local clearances for those 8 pads - Added more silkscreen/rotated all existing silkscreen to face one way
Parts:
- added D1: PWR LED, mod:LTST-C191KGKT, symbol Device:LED
- added D2: LED4, mod:LTST-C191KGKT, symbol Device:LED
- added D3: LED3, mod:LTST-C191KGKT, symbol Device:LED
- added D4: LED2, mod:LTST-C191KGKT, symbol Device:LED
- added D5: LED1, mod:LTST-C191KGKT, symbol Device:LED
- added R10, R11, R7, R8, R9: 68Ω, mod:ERJ-3EKF10R0V, symbol Device:R_Small_US
Connections:
- wire segments 199 -> 209
- no-connect marks 29 -> 25

Commit message: - Changed PIC from MR to PT package for ease of soldering - Increased size from 2"-1.2"
Parts:
- removed U1: PIC32MX340F512H-80I_MR, mod:PIC32MX340F512H-80I&slash_MR, symbol 2020-10-30_02-35-18:PIC32MX340F512H-80I_MR
- added U1: PIC32MX340F512H-80V_PT, mod:PIC32MX340F512H-80V&slash_PT, symbol ul_PIC32MX340F512H80VPT:PIC32MX340F512H-80V_PT
Connections:
- no-connect marks 25 -> 24
Other:
- moved on the sheet: C5

Commit message: Made a few changes for boardhouse - Moved title silkscreen up like 10mil - Shifted mount holes from vias to an actual footprint
Parts:
- added H1, H2, H3, H4: MountingHole_Pad, mod:test, symbol Mechanical:MountingHole_Pad
Changed lines of the file:
@@
 	9600 5150 9600 5950
 NoConn ~ 9500 5050
+$Comp
+L Mechanical:MountingHole_Pad H4
+U 1 1 5FA5E786
+P 11150 600
+F 0 "H4" H 10900 650 50  0000 L CNN
+F 1 "MountingHole_Pad" H 10400 550 50  0000 L CNN
+F 2 "mod:test" H 11150 600 50  0001 C CNN
+F 3 "~" H 11150 600 50  0001 C CNN
+	1    11150 600
+	1    0    0    -1
+$EndComp
+$Comp
+L Mechanical:MountingHole_Pad H3
+U 1 1 5FA5F9BF
+P 11100 6300
+F 0 "H3" H 10900 6400 50  0000 L CNN
+F 1 "MountingHole_Pad" H 10300 6300 50  0000 L CNN
+F 2 "mod:test" H 11100 6300 50  0001 C CNN
+F 3 "~" H 11100 6300 50  0001 C CNN
+	1    11100 6300
+	1    0    0    -1
+$EndComp
+$Comp
+L power:GNDREF #PWR026
+U 1 1 5FA6206F
+P 550 700
+F 0 "#PWR026" H 550 450 50  0001 C CNN
+F 1 "GNDREF" H 650 550 50  0000 C CNN
+F 2 "" H 550 700 50  0001 C CNN
+F 3 "" H 550 700 50  0001 C CNN
+	1    550  700
+	1    0    0    -1
+$EndComp
+$Comp
+L Mechanical:MountingHole_Pad H1
+U 1 1 5FA5E21B
+P 550 600
+F 0 "H1" H 650 649 50  0000 L CNN
+F 1 "MountingHole_Pad" H 650 558 50  0000 L CNN
+F 2 "mod:test" H 550 600 50  0001 C CNN
+F 3 "~" H 550 600 50  0001 C CNN
+	1    550  600
+	1    0    0    -1
+$EndComp
+$Comp
+L power:GNDREF #PWR029
+U 1 1 5FA6E512
+P 11150 700
+F 0 "#PWR029" H 11150 450 50  0001 C CNN
+F 1 "GNDREF" H 11050 550 50  0000 C CNN
+F 2 "" H 11150 700 50  0001 C CNN
+F 3 "" H 11150 700 50  0001 C CNN
+	1    11150 700
+	1    0    0    -1
+$EndComp
+$Comp
+L power:GNDREF #PWR028
+U 1 1 5FA6FBB2
+P 11100 6400
+F 0 "#PWR028" H 11100 6150 50  0001 C CNN
+F 1 "GNDREF" H 10900 6350 50  0000 C CNN
+F 2 "" H 11100 6400 50  0001 C CNN
+F 3 "" H 11100 6400 50  0001 C CNN
+	1    11100 6400
+	1    0    0    -1
+$EndComp
+$Comp
+L power:GNDREF #PWR027
+U 1 1 5FA7C00B
+P 650 6400
+F 0 "#PWR027" H 650 6150 50  0001 C CNN
+F 1 "GNDREF" H 655 6227 50  0000 C CNN
+F 2 "" H 650 6400 50  0001 C CNN
+F 3 "" H 650 6400 50  0001 C CNN
+	1    650  6400
+	1    0    0    -1
+$EndComp
+$Comp
+L Mechanical:MountingHole_Pad H2
+U 1 1 5FA60A4E
+P 650 6300
+F 0 "H2" H 750 6349 50  0000 L CNN
+F 1 "MountingHole_Pad" H 750 6258 50  0000 L CNN
+F 2 "mod:test" H 650 6300 50  0001 C CNN
+F 3 "~" H 650 6300 50  0001 C CNN
+	1    650  6300
+	1    0    0    -1
+$EndComp
 $EndSCHEMATC

Commit message: - Began work on dev board V2
Parts:
- removed C1: 0.1uF, mod:CL10A106MQ8NNNC, symbol pspice:C
- removed J1: ICSP, mod:01x06, symbol Connector:Conn_01x06_Female
- removed J4: 3.3v VDD, mod:RESC3115X65N, symbol Connector_Generic:Conn_01x02
- removed J5: VSS, mod:RESC3115X65N, symbol Connector_Generic:Conn_01x02
- removed J6: GPIO Header, mod:02x20, symbol Connector_Generic:Conn_02x10_Odd_Even
- removed R1, R2: 470Ω, mod:ERJ-3EKF10R0V, symbol Device:R_Small_US
- added C10, C9: C, mod:0603, symbol pspice:C
- added C4, C5, C6: 1uF, mod:0603, symbol pspice:C
- added J1: Analog GPIO, mod:02x05, symbol Connector_Generic:Conn_01x10
- added J2: ICSP, mod:01x06, symbol Connector_Generic:Conn_01x06
- added J5: USB4085-GF-A_REVA, mod:GCT_USB4085-GF-A_REVA, symbol USB4085-GF-A_REVA:USB4085-GF-A_REVA
- added J6: Digital GPIO, mod:02x20, symbol Connector_Generic:Conn_01x20
- added J8: Power, mod:01x06, symbol Connector_Generic:Conn_01x06
- added R12, R13: R, mod:0603, symbol Device:R_Small_US
- added R8, R9: 5.1kΩ, mod:0603, symbol Device:R_Small_US
- added U2: AZ1117EH-3.3TRG1, mod:SOT230P700X180-4N, symbol AZ1117EH-3.3TRG1:AZ1117EH-3.3TRG1
- added U3: AZ1117EH-5.0TRG1, mod:SOT230P700X180-4N, symbol AZ1117EH-5.0TRG1:AZ1117EH-5.0TRG1
- added Y1: Y, mod:9B-8.000MAAJ-B, symbol Device:Crystal
- C1: renamed from C2; footprint mod:CL10A106MQ8NNNC -> mod:0603; Mfr (none) -> Samsung Electro-Mechanics; Mfr # (none) -> CL10B104KA8NNNC
- C2: renamed from C3; footprint mod:CL10A106MQ8NNNC -> mod:0603; Mfr (none) -> Samsung Electro-Mechanics; Mfr # (none) -> CL10B104KA8NNNC
- C3: renamed from C4; footprint mod:CL10A106MQ8NNNC -> mod:0603; Mfr (none) -> Samsung Electro-Mechanics; Mfr # (none) -> CL10B104KA8NNNC
- C7: renamed from C6; footprint mod:CL10A106MQ8NNNC -> mod:0603; Mfr (none) -> Samsung Electro-Mechanics; Mfr # (none) -> CL10A106MQ8NNNC
- C8: renamed from C5; footprint mod:CL10A106MQ8NNNC -> mod:0603; Mfr (none) -> Samsung Electro-Mechanics; Mfr # (none) -> CL10B104KA8NNNC
- D1, D2, D3, D4, D5: footprint mod:LTST-C191KGKT -> mod:0603
- H1, H2, H3, H4: footprint mod:test -> mod:#6
- R1: renamed from R7; footprint mod:ERJ-3EKF10R0V -> mod:0603
- R10: renamed from R5; footprint mod:ERJ-3EKF10R0V -> mod:0603; Mfr (none) -> Stackpole Electronics Inc; Mfr # (none) -> RMCF0603FT4K70
- R11: renamed from R6; footprint mod:ERJ-3EKF10R0V -> mod:0603; Mfr (none) -> Stackpole Electronics Inc; Mfr # (none) -> RMCF0603FT4K70
- R2: renamed from R8; footprint mod:ERJ-3EKF10R0V -> mod:0603
- R3: footprint mod:ERJ-3EKF10R0V -> mod:0603; Mfr (none) -> Stackpole Electronics Inc; Mfr # (none) -> RMCF0603FT10K0
- R4: renamed from R9; footprint mod:ERJ-3EKF10R0V -> mod:0603
- R5: renamed from R10; footprint mod:ERJ-3EKF10R0V -> mod:0603
- R6: renamed from R4; footprint mod:ERJ-3EKF10R0V -> mod:0603; Mfr (none) -> Stackpole Electronics Inc; Mfr # (none) -> RMCF0603FT10R0
- R7: renamed from R11; footprint mod:ERJ-3EKF10R0V -> mod:0603
- renumbered J2 to J3, J3 to J4
Connections:
- net labels added: +5V, VCC
- wire segments 209 -> 286
- no-connect marks 24 -> 12
Other:
- moved on the sheet: C1, C2, C3, C7, C8, D1, D2, D3, D4, D5, J3, J4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

Commit message: Finished following changes... - Removed SMD test points for power and replaced with USB-C port - Added 2 voltage regulators for 5v and 3v3 - Added a 6 port power header for 5v, 3v3, GND, and VIN - Added a 10 port analog header - Shifted ICSP PGD and PGC pins from the 1st to 2nd set to allow for use of AN0 and AN1 which are also used for possible reference voltages for analog data - Added a crystal oscillator - Simplified MCLR circuit, think there was a lot more there than was necessary
Parts:
- removed H1, H2, H3, H4: MountingHole_Pad, mod:#6, symbol Mechanical:MountingHole_Pad
- C1, C10, C2, C3, C4, C5, C6, C7, C8, C9: symbol pspice:C -> test-rescue:C-pspice
- J1: value Analog GPIO -> Analog
- J6: value Digital GPIO -> Digital
Connections:
- net GNDREF: now also J3.4 (Pin_4)
- net at J5.B6 (DP2): now also J5.B7 (DN2)
- no-connect marks 12 -> 11
Changed lines of the file:
@@
 Sheet 1 1
 Title "PIC32MX Dev Board"
-Date "2020-11-05"
-Rev "4"
+Date "2020-11-24"
+Rev "5"
 Comp ""
 Comment1 ""
@@
 Wire Wire Line
 	4450 1850 4400 1850
-NoConn ~ 4400 1950
 NoConn ~ 3900 2550
 NoConn ~ 3900 2650
@@
 $EndComp
 $Comp
-L pspice:C C7
+L test-rescue:C-pspice C7
 U 1 1 5FD9384F
 P 8300 3650
@@
 	2600 3750 3600 3750
 $Comp
-L pspice:C C3
+L test-rescue:C-pspice C3
 U 1 1 5FA6CD8B
 P 3500 4400
@@
 	3100 4250 3200 4250
 $Comp
-L pspice:C C2
+L test-rescue:C-pspice C2
 U 1 1 5FD77597
 P 3450 5000
@@
 	3450 3300 3450 3250
 $Comp
-L pspice:C C1
+L test-rescue:C-pspice C1
 U 1 1 5FA64A53
 P 3450 3400
@@
 U 1 1 5FA522C7
 P 3300 4250
-F 0 "R6" V 3507 4250 50  0000 C CNN
-F 1 "10Ω" V 3416 4250 50  0000 C CNN
+F 0 "R6" V 3400 4300 50  0000 C CNN
+F 1 "10Ω" V 3400 4150 50  0000 C CNN
 F 2 "mod:0603" V 3230 4250 50  0001 C CNN
 F 3 "~" H 3300 4250 50  0001 C CNN
@@
 P 9100 3100
 F 0 "J6" H 9180 3092 50  0000 L CNN
-F 1 "Digital GPIO" H 9180 3001 50  0000 L CNN
+F 1 "Digital" H 9180 3001 50  0000 L CNN
 F 2 "mod:02x20" H 9100 3100 50  0001 C CNN
 F 3 "~" H 9100 3100 50  0001 C CNN
@@
 	8500 1450 8600 1450
 Connection ~ 7700 1600
-Connection ~ 8600 1450
-Wire Wire Line
-	8600 1450 8600 1550
 $Comp
 L AZ1117EH-5.0TRG1:AZ1117EH-5.0TRG1 U3
@@
 	1    6600 1300
 	-1   0    0    1
-$EndComp
-$Comp
-L power:GNDREF #PWR029
-U 1 1 600C24E5
-P 8600 1550
-F 0 "#PWR029" H 8600 1300 50  0001 C CNN
-F 1 "GNDREF" V 8605 1422 50  0001 R CNN
-F 2 "" H 8600 1550 50  0001 C CNN
-F 3 "" H 8600 1550 50  0001 C CNN
-	1    8600 1550
-	1    0    0    -1
 $EndComp
 $Comp
@@
 P 1850 4650
 F 0 "J1" H 2150 4900 50  0000 C CNN
-F 1 "Analog GPIO" H 2150 4800 50  0000 C CNN
+F 1 "Analog" H 2150 4800 50  0000 C CNN
 F 2 "mod:02x05" H 1850 4650 50  0001 C CNN
 F 3 "~" H 1850 4650 50  0001 C CNN
@@
 Connection ~ 6200 1400
 $Comp
-L pspice:C C6
+L test-rescue:C-pspice C6
 U 1 1 604CCE88
 P 7100 1300
@@
 Connection ~ 5150 1550
 $Comp
-L pspice:C C4
+L test-rescue:C-pspice C4
 U 1 1 60457AC1
 P 5050 1550
@@
 Connection ~ 6050 1400
 $Comp
-L pspice:C C5
+L test-rescue:C-pspice C5
 U 1 1 60441459
 P 6050 1300
@@
 $EndComp
 $Comp
-L pspice:C C10
+L test-rescue:C-pspice C10
 U 1 1 5FE82939
 P 9850 5000
@@
 $EndComp
 $Comp
-L pspice:C C9
+L test-rescue:C-pspice C9
 U 1 1 5FE7EDE4
 P 9850 4700
@@
 Wire Wire Line
 	8000 1450 8000 1400
-$Comp
-L power:GNDREF #PWR039
-U 1 1 5FA6FBB2
-P 11100 6400
-F 0 "#PWR039" H 11100 6150 50  0001 C CNN
-F 1 "GNDREF" H 10900 6350 50  0001 C CNN
-F 2 "" H 11100 6400 50  0001 C CNN
-F 3 "" H 11100 6400 50  0001 C CNN
-	1    11100 6400
-	1    0    0    -1
-$EndComp
-$Comp
-L Mechanical:MountingHole_Pad H3
-U 1 1 5FA5F9BF
-P 11100 6300
-F 0 "H3" H 10900 6400 50  0000 L CNN
-F 1 "MountingHole_Pad" H 10300 6300 50  0000 L CNN
-F 2 "mod:#6" H 11100 6300 50  0001 C CNN
-F 3 "~" H 11100 6300 50  0001 C CNN
-	1    11100 6300
-	1    0    0    -1
-$EndComp
-$Comp
-L power:GNDREF #PWR040
-U 1 1 5FA6E512
-P 11150 700
-F 0 "#PWR040" H 11150 450 50  0001 C CNN
-F 1 "GNDREF" H 11050 550 50  0001 C CNN
-F 2 "" H 11150 700 50  0001 C CNN
-F 3 "" H 11150 700 50  0001 C CNN
-	1    11150 700
-	1    0    0    -1
-$EndComp
-$Comp
-L Mechanical:MountingHole_Pad H4
-U 1 1 5FA5E786
-P 11150 600
-F 0 "H4" H 10900 650 50  0000 L CNN
-F 1 "MountingHole_Pad" H 10400 550 50  0000 L CNN
-F 2 "mod:#6" H 11150 600 50  0001 C CNN
-F 3 "~" H 11150 600 50  0001 C CNN
-	1    11150 600
-	1    0    0    -1
-$EndComp
-$Comp
-L Mechanical:MountingHole_Pad H2
-U 1 1 5FA60A4E
-P 650 6300
-F 0 "H2" H 750 6349 50  0000 L CNN
-F 1 "MountingHole_Pad" H 750 6258 50  0000 L CNN
-F 2 "mod:#6" H 650 6300 50  0001 C CNN
-F 3 "~" H 650 6300 50  0001 C CNN
-	1    650  6300
-	1    0    0    -1
-$EndComp
-$Comp
-L power:GNDREF #PWR02
-U 1 1 5FA7C00B
-P 650 6400
-F 0 "#PWR02" H 650 6150 50  0001 C CNN
-F 1 "GNDREF" H 655 6227 50  0001 C CNN
-F 2 "" H 650 6400 50  0001 C CNN
-F 3 "" H 650 6400 50  0001 C CNN
-	1    650  6400
-	1    0    0    -1
-$EndComp
-$Comp
-L Mechanical:MountingHole_Pad H1
-U 1 1 5FA5E21B
-P 550 600
-F 0 "H1" H 650 649 50  0000 L CNN
-F 1 "MountingHole_Pad" H 650 558 50  0000 L CNN
-F 2 "mod:#6" H 550 600 50  0001 C CNN
-F 3 "~" H 550 600 50  0001 C CNN
-	1    550  600
-	1    0    0    -1
-$EndComp
-$Comp
-L power:GNDREF #PWR01
-U 1 1 5FA6206F
-P 550 700
-F 0 "#PWR01" H 550 450 50  0001 C CNN
-F 1 "GNDREF" H 650 550 50  0001 C CNN
-F 2 "" H 550 700 50  0001 C CNN
-F 3 "" H 550 700 50  0001 C CNN
-	1    550  700
-	1    0    0    -1
-$EndComp
 $Comp
 L Device:LED D1
@@
 $EndComp
 $Comp
-L pspice:C C8
+L test-rescue:C-pspice C8
 U 1 1 5FD89C95
 P 8400 5000
@@
 	-1   0    0    1
 $EndComp
+Wire Wire Line
+	7900 1400 7900 1500
+Wire Wire Line
+	7900 1500 8100 1500
+Wire Wire Line
+	8100 1500 8100 1400
+Connection ~ 8600 1450
+$Comp
+L power:GNDREF #PWR029
+U 1 1 600C24E5
+P 8600 1550
+F 0 "#PWR029" H 8600 1300 50  0001 C CNN
+F 1 "GNDREF" V 8605 1422 50  0001 R CNN
+F 2 "" H 8600 1550 50  0001 C CNN
+F 3 "" H 8600 1550 50  0001 C CNN
+	1    8600 1550
+	1    0    0    -1
+$EndComp
+Wire Wire Line
+	8600 1450 8600 1550
+$Comp
+L power:GNDREF #PWR0101
+U 1 1 5FE6521B
+P 4550 1950
+F 0 "#PWR0101" H 4550 1700 50  0001 C CNN
+F 1 "GNDREF" V 4555 1822 50  0001 R CNN
+F 2 "" H 4550 1950 50  0001 C CNN
+F 3 "" H 4550 1950 50  0001 C CNN
+	1    4550 1950
+	1    0    0    -1
+$EndComp
+Wire Wire Line
+	4400 1950 4550 1950
 $EndSCHEMATC

Commit message: - added pic32 mfr and mfr # because why not
Parts:
- U1: Mfr (none) -> Microchip Technology; Mfr # (none) -> PIC32MX340F512H
Changed lines of the file:
@@
 F 2 "mod:PIC32MX340F512H-80V&slash_PT" H 6000 2790 60  0001 C CNN
 F 3 "" H 3900 2550 60  0000 C CNN
+F 4 "Microchip Technology" H 1000 2550 50  0001 C CNN "Mfr"
+F 5 "PIC32MX340F512H" H 1000 2550 50  0001 C CNN "Mfr #"
 	1    1000 2550
 	1    0    0    -1
